Commit message: modify model

File: w1bot_description/urdf/w1bot.xacro (robot description, xacro)
@@ -1,13 +1,15 @@
 <?xml version="1.0"?>
 <robot xmlns:xacro="http://www.ros.org/wiki/xacro" name="w1bot">
-  <xacro:property name="base_width" value="0.16"/>
-  <xacro:property name="base_len" value="0.16"/>
-  <xacro:property name="wheel_radius" value="0.035"/>
+  <xacro:property name="base_width" value="0.21"/>
+  <xacro:property name="base_len" value="0.21"/>
+  <xacro:property name="wheel_radius" value="0.0525"/>
   <xacro:property name="base_wheel_gap" value="0.007"/>
-  <xacro:property name="wheel_separation" value="0.15"/>
-  <xacro:property name="wheel_joint_offset" value="0.02"/>
-  <xacro:property name="caster_wheel_radius" value="${wheel_radius/2}"/>
+  <xacro:property name="wheel_separation" value="0.25"/>
+  <xacro:property name="wheel_joint_x_offset" value="0.0"/>
+  <xacro:property name="wheel_joint_z_offset" value="0.02"/>
+  <xacro:property name="caster_wheel_radius" value="0.008"/>
   <xacro:property name="caster_wheel_mass" value="0.001"/>
-  <xacro:property name="caster_wheel_joint_offset" value="-0.052"/>
+  <xacro:property name="caster_wheel_joint_offset" value="0.105"/>
+  <xacro:property name="caster_wheel_joint_z_offset" value="0.025"/>
   <xacro:include filename="$(find w1bot_description)/urdf/w1bot_gazebo_plugins.xacro" />
   <!--Color Properties-->
@@ -96,5 +98,5 @@
       <parent link="base_link"/>
       <child link="${prefix}_wheel"/>
-      <origin xyz="${wheel_joint_offset} ${((base_width/2)+base_wheel_gap)*reflect} -0.005" rpy="0 0 0"/>
+      <origin xyz="${wheel_joint_x_offset} ${((base_width/2)+base_wheel_gap)*reflect} ${wheel_joint_z_offset}" rpy="0 0 0"/>
     </joint>
   </xacro:macro>
@@ -102,6 +104,6 @@
   <xacro:wheel prefix="left" reflect="1"/>
   <xacro:wheel prefix="right" reflect="-1"/>
-  <!--Caster Wheel Link-->
-  <link name="caster_wheel">
+  <!--Caster Front Wheel Link-->
+  <link name="caster_front_wheel">
     <visual>
       <origin xyz="0 0 0" rpy="0 0 0"/>
@@ -119,10 +121,34 @@
     <xacro:sphere_inertia m="1" r="${caster_wheel_radius}"/>
   </link>
-  <!--Caster Wheel Joint-->
-  <joint name="caster_wheel_joint" type="continuous">
+  <!--Caster Front Wheel Joint-->
+  <joint name="caster_front_wheel_joint" type="continuous">
     <axis xyz="0 1 0" rpy="0 0 0" />
     <parent link="base_link"/>
-    <child link="caster_wheel"/>
-    <origin xyz="${caster_wheel_joint_offset} 0 -${caster_wheel_radius+0.005}" rpy="0 0 0"/>
+    <child link="caster_front_wheel"/>
+    <origin xyz="-${caster_wheel_joint_offset} 0 -${caster_wheel_joint_z_offset}" rpy="0 0 0"/>
+  </joint>
+<!--Caster Rear Wheel Link-->
+  <link name="caster_rear_wheel">
+    <visual>
+      <origin xyz="0 0 0" rpy="0 0 0"/>
+      <geometry>
+        <sphere radius="${caster_wheel_radius}"/>
+      </geometry>
+      <material name="blue"/>
+    </visual>
+    <collision>
+      <origin xyz="0 0 0" rpy="0 0 0"/>
+      <geometry>
+        <sphere radius="${caster_wheel_radius}"/>
+      </geometry>
+    </collision>
+    <xacro:sphere_inertia m="1" r="${caster_wheel_radius}"/>
+  </link>
+  <!--Caster Rear Wheel Joint-->
+  <joint name="caster_rear_wheel_joint" type="continuous">
+    <axis xyz="0 1 0" rpy="0 0 0" />
+    <parent link="base_link"/>
+    <child link="caster_rear_wheel"/>
+    <origin xyz="${caster_wheel_joint_offset} 0 -${caster_wheel_joint_z_offset}" rpy="0 0 0"/>
   </joint>
 </robot>
